Commit message: gripper mesh has longer tip

File: urdf/edo_gripper_dummy.xacro (robot description, xacro)
@@ -43,5 +43,5 @@
             <parent link="${robot_prefix}_gripper_link"/>
             <child link="${robot_prefix}_gripper_left_base_link"/>
-            <origin xyz="0 0.025 0.0195" rpy="${PI / 2} 0 ${PI / 2}"/>
+            <origin xyz="0 0.025 0.0195" rpy="${(PI / 2)} -0.5 ${PI / 2}"/>
             <axis xyz="0 0 1"/>
             <limit lower="${-PI / 2}" upper="${PI / 2}"
@@ -79,5 +79,5 @@
             <parent link="${robot_prefix}_gripper_left_base_link"/>
             <child link="${robot_prefix}_gripper_left_finger_link"/>
-            <origin xyz="0 0.04 0" rpy="0 0 0"/>
+            <origin xyz="0 0.04 0" rpy="0 0 -0.5"/>
             <axis xyz="0 0 1"/>
             <limit lower="${-PI / 2}" upper="${PI / 2}"
@@ -115,5 +115,5 @@
             <parent link="${robot_prefix}_gripper_link"/>
             <child link="${robot_prefix}_gripper_right_base_link"/>
-            <origin xyz="0 -0.025 0.0195" rpy="${PI / 2} 0 -${PI / 2}"/>
+            <origin xyz="0 -0.025 0.0195" rpy="${PI / 2} -0.5 -${PI / 2}"/>
             <axis xyz="0 0 1"/>
             <limit lower="${-PI / 2}" upper="${PI / 2}"
@@ -151,5 +151,5 @@
             <parent link="${robot_prefix}_gripper_right_base_link"/>
             <child link="${robot_prefix}_gripper_right_finger_link"/>
-            <origin xyz="0 0.04 0" rpy="0 0 0"/>
+            <origin xyz="0 0.04 0" rpy="0 0 -0.5"/>
             <axis xyz="0 0 1"/>
             <limit lower="${-PI / 2}" upper="${PI / 2}"
